File: hardware/osd.kicad_sch (KiCad schematic)
At the start: 21 parts, among them U10 SN74LVC1G3157DTBR, U11 COS8051SOT, U12 TLV7031DPWR

Commit message: ok
Parts:
- R36, R37: MPN (none) -> RC0201FR-07510RL; Manufacturer (none) -> YAGEO
- TP1, TP2, TP3, TP4: now left out of the parts list
