File: hardware/power.kicad_sch (KiCad schematic)
At the start: 34 parts, among them U3 TI LMR51430YFDDCR, U4 TI LMR51430YFDDCR, U5 TPS2116DRLR, U6 NCV8187AMT180TAG, U7 LP5912-3.3DRVR

Commit message: ok
Parts:
- removed C28: 4.7uF, Capacitor_SMD:C_0402_1005Metric, symbol Device:C
- removed C29: 100n, Capacitor_SMD:C_0201_0603Metric, symbol Device:C
- removed D2, D3: RB161QS-40_C28646385, lib:SOD-882_L1.0-W0.6-RD, symbol lib:RB161QS-40_C28646385
- removed D6: LED_1_Green, LED_SMD:LED_0402_1005Metric, symbol Device:LED
- removed R19: 100k, Resistor_SMD:R_0201_0603Metric, symbol Device:R
- removed R20: 39k, Resistor_SMD:R_0201_0603Metric, symbol Device:R
- removed R27: 2.4k, Resistor_SMD:R_0201_0603Metric, symbol Device:R
- removed U3, U4: TI LMR51430YFDDCR, lib:SOT-23-6_L2.9-W1.6-P0.95-LS2.9-BL, symbol lib:LMR51420YDDCR
- removed U5: TPS2116DRLR, lib:SOT-583-8_L2.1-W1.6-P0.50-LS1.6-BL, symbol lib:TPS2116DRLR
- removed U6: NCV8187AMT180TAG, lib:WDFN-6_L2.0-W2.0-P0.65-BL-EP, symbol lib:NCV8187AMT180TAG
- added C42: 22uF, Capacitor_SMD:C_0402_1005Metric, symbol Device:C
- added D10, D6: DSK24, lib:SOD-123_L2.8-W1.8-LS3.7-RD, symbol lib:DSK24_C64890
- added D9: LED_1_Green, LED_SMD:LED_0402_1005Metric, symbol Device:LED
- added R39: 6.49k, Resistor_SMD:R_0201_0603Metric, symbol Device:R
- added U15: LP5912-1.8DRVR, lib:WSON-6-1EP_2x2mm_P0.65mm_EP1x1.6mm_ThermalVias, symbol lib:LP5912-1.8DRVR
- added U16, U6: LMR51635YDDCR, lib:SOT-23-6_L2.9-W1.6-P0.95-LS2.8-BL, symbol lib:LMR51635YDDCR
- C31: value 22uF -> 4.7uF; LCSC C105226 -> C23733; MPN CL05A226MQ5QUNC -> CL05A475MP5NRNC
- D4, D5, D7: MPN XL-1005UGC -> XL-1005UGC
- R22: value 6.49k -> 8.87k; LCSC C2107920 -> C332577; MPN (none) -> RTT018871FTH; Manufacturer (none) -> RALEC
- R24: value 13.7k -> 19.1k; LCSC C320695 -> C320741; MPN RC-01W1372FT -> RC-01W1912FT
- R25: MPN (none) -> RC0201FR-077K5L; Manufacturer (none) -> YAGEO
- R26: MPN (none) -> RTT012401FTH; Manufacturer (none) -> RALEC
- R28: MPN (none) -> RC0201FR-07510RL; Manufacturer (none) -> YAGEO
Connections:
- net +5V_BUCK is gone; now on net +5V: C27.1, L3.2, R23.2, R26.1
- net +1.8V_GYRO: now also C42.1, U15.1 (OUT); no longer C31.1
- net +5V: now also D6.2 (A); no longer C30.1, U7.4 (EN), U7.6 (IN)
- net +5V_USB: now also D10.2 (A)
- net +BATT: now also U16.2 (EN), U16.3 (VIN), U6.3 (VIN)
- net 1.8V_PG: now also D9.2 (A), R39.2, U15.3 (PG)
- net 10V_ENABLE: now also U6.2 (EN)
- net GND: now also C42.2, D9.1 (K), U15.5 (GND), U15.7 (EP), U16.4 (GND), U6.4 (GND)
- net at R21.1, R22.1: now also U6.1 (FB)
- net at R23.1, R24.1: now also U16.1 (FB)
- net at C24.1, L2.1: now also U6.5 (SW)
- net at C24.2: now also U6.6 (CB)
- net at C25.1, L3.1: now also U16.5 (SW)
- net at C25.2: now also U16.6 (CB)
- new net +4v5: C30.1, C31.1, D10.1 (K), D6.1 (K), R39.1, U15.4 (EN), U15.6 (IN), U7.4 (EN), U7.6 (IN)
Other:
- note added: "10V (3.5A)"
- note added: "10V: Vout = Vref × (1 + R_top / R_bottom) = 0.8 × (1 + 100 / 8.87) = 0.8 × 12.274 = 9.819 V"
- note added: "4.3 - 60V input Synchronous buck 1.1MHz"
- note added: "5V (3.5A)"
- note added: "5V: Vout = Vref × (1 + R_top / R_bottom) = 0.8 × (1 + 100 / 19.1) = 0.8 × 6.236 = 4.988 V"
- note added: "PFM version of the LMR51635 for better light-load efficiency and spread-spectrum EMI, at the cost of variable switching frequency at light load"
- note removed: "1.2A is way too much, but anyway PSSR of 80dB!!! until 10kHz Power Good output for LED"
- note removed: "10V (2A)"
- note removed: "4.5 - 36V input Synchronous buck 1.1MHz"
- note removed: "5V (2A)"
- note removed: "FPWM version of the LMR51430 for less output ripple at low voltage and more consistency but less efficient"
- note removed: "LMR51430 = 3A output LMR51420 = 2A output (pin compatible)"
- note removed: "Vout = Vref × (1 + R_top / R_bottom) = 0.6 × (1 + 100 / 13.7) = 0.6 × 8.299 = 4.980 V"
- note removed: "Vout = Vref × (1 + R_top / R_bottom) = 0.6 × (1 + 100 / 6.49) = 0.6 × 16.408 = 9.845 V"
- note removed: "max 30mA on PG (open collector/drain), datasheet assumes 6mA for a typical application"
