File: hardware/rp2350a.kicad_sch (KiCad schematic)
At the start: 48 parts, among them Q1 AP1606, Q2 AP1606, U1 TS2306A 240GF MSM 9_C2976675, U2 RP2354B_C39843328, X1 XTM25012000JT00351001

Commit message: ok
Parts:
- R18: MPN (none) -> RTT012401FTH; Manufacturer (none) -> RALEC
Connections:
- net +5V renamed +4v5
